File: Hardware/PCB/IMPASS/sensorres.kicad_sch (KiCad schematic)
At the start: 21 parts, among them J13 SENSORES, U2 ACS712xLCTR-30A, U3 ACS712xLCTR-30A, U4 ACS712xLCTR-30A, U5 ACS712xLCTR-30A, U6 ACS712xLCTR-30A, U7 ACS712xLCTR-30A, U8 LM75B, U9 LM75B

Commit message: IMPASS schematics update
Parts:
- added C11, C12, C13, C14, C15, C16: 1nF, Capacitor_SMD:C_0603_1608Metric, symbol Device:C
Connections:
- net GND1: now also C11.2, C12.2, C13.2, C14.2, C15.2, C16.2
- net at U7.6 (FILTER): now also C14.1
- net at U6.6 (FILTER): now also C15.1
- net at U3.6 (FILTER): now also C12.1
- net at U2.6 (FILTER): now also C11.1
- net at U4.6 (FILTER): now also C13.1
