File: Hardware/PCB/IMPASS/sensorres.kicad_sch (KiCad schematic)
At the start: 31 parts, among them J13 SENSORES, U12 MPU-6050, U2 ACS712xLCTR-30A, U3 ACS712xLCTR-30A, U4 ACS712xLCTR-30A, U5 ACS712xLCTR-30A, U6 ACS712xLCTR-30A, U7 ACS712xLCTR-30A, U8 LM75B, U9 AS5047D

Commit message: Update to v1
Parts:
- removed U12: MPU-6050, Sensor_Motion:InvenSense_QFN-24_4x4mm_P0.5mm, symbol Sensor_Motion:MPU-6050
- added C20, C21, C22, C23, C24, C25, C26: 100nF, Capacitor_SMD:C_0603_1608Metric, symbol Device:C
- added C27: 1uF, Capacitor_SMD:C_0603_1608Metric, symbol Device:C
- added U12: MCP3008, Package_SO:SOIC-16_3.9x9.9mm_P1.27mm, symbol Analog_ADC:MCP3008
- added U13: LM75B, Package_SO:SOIC-8_3.9x4.9mm_P1.27mm, symbol Sensor_Temperature:LM75B
- C18: value 2.2nF -> 100nF
Connections:
- net 3.3V is gone; now on net 5V_in: C19.1
- net +5VA: now also C20.1, C21.1, C22.1, C23.1, C24.1, C25.1, C26.1
- net GND1: now also C20.2, C21.2, C22.2, C23.2, C24.2, C25.2, C26.2
- net GND_in: now also U9.13 (GND), U9.5 (TST), C27.2, U12.14 (AGND), U12.9 (DGND), U13.4 (GND)
- net SCL: now also U13.2 (SCL)
- net SDA: now also U13.1 (SDA)
- net 5V_in: now reaches C18.1
- net 5V_in: now also C17.1, U9.11 (VDD), U12.15 (Vref), U12.16 (Vdd), U13.5 (A2), U13.6 (A1), U13.7 (A0), U13.8 (+Vs)
- net CS_INCL: now reaches U9.1 (~{CS})
- net at U9.12 (VDD3V3): now also C27.1
- net SCK: now reaches U9.2 (CLK)
- net SCK: now also U12.13 (CLK)
- net MISO: now reaches U9.3 (MISO)
- net MISO: now also U12.12 (Dout)
- net MOSI: now reaches U9.4 (MOSI)
- net MOSI: now also U12.11 (Din)
- new net ADC1: U12.1 (CH0)
- new net ADC2: U12.2 (CH1)
- new net ADC3: U12.3 (CH2)
- new net ADC4: U12.4 (CH3)
- new net ADC5: U12.5 (CH4)
- new net ADC6: U12.6 (CH5)
- new net CS_ADC: U12.10 (~{CS}/SHDN)
- no-connect marks 3 -> 10
Other:
- moved on the sheet: C11, C12, C13, C14, C15, C16, D1, D2, D3, D4, D5, D6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

Commit message: Update v1
Other:
- note added: "Sensores de la placa Lógica"
- note added: "Sensores del SHIELD"
- company: (none) -> Luis Miguel Carmona Cortés
- title: (none) -> IMPASS 
- moved on the sheet: C11, C12, C13, C14, C15, C16, C18, C19, C20, C21, C22, C23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
