File: Hardware/PCB/IMPASS/IMPASS.kicad_pcb (KiCad board)
At the start: 2 copper layers, 80 x 100 mm, 142 parts, among them J1 PUENTE H, J10 SENSORES, J11 SOLENOIDES, J12 POWER, J13 SENSORES, J14 SOLENOIDES, J15 PUENTE H, J16 PUENTE H, J2 POWER, J3 EJE1, J4 EJE2, J5 EJE3, J6 VM, J7 PUENTE H, J8 SOLENOIDES, J9 PROG, Q1 DMN3008SFG, Q10 DMN3008SFG, Q11 DMN3008SFG, Q12 DMN3008SFG, Q13 DMN3008SFG, Q14 DMN3008SFG, Q15 DMN3008SFG, Q16 DMN3008SFG, Q17 DMN3008SFG, Q18 DMN3008SFG, Q19 DMN3008SFG, Q2 DMN3008SFG, Q20 DMN3008SFG, Q21 DMN3008SFG, Q22 DMN3008SFG, Q23 DMN3008SFG, Q24 DMN3008SFG, Q25 2N7002, Q26 2N7002, Q27 2N7002, Q28 2N7002, Q29 2N7002, Q3 DMN3008SFG, Q30 2N7002, Q31 2N7002, Q32 2N7002, Q33 2N7002, Q34 2N7002, Q35 2N7002, Q36 2N7002, Q37 2N7002, Q38 2N7002, Q39 2N7002, Q4 DMN3008SFG, Q40 2N7002, Q41 2N7002, Q42 2N7002, Q43 DMN3008SFG, Q44 DMN3008SFG, Q45 DMN3008SFG, Q46 2N7002, Q47 2N7002, Q48 2N7002, Q5 DMN3008SFG, Q6 DMN3008SFG, Q7 DMN3008SFG, Q8 DMN3008SFG, Q9 DMN3008SFG, SW1 RESET, SW2 BOOT, U1 ESP32-S3-WROOM-1, U10 AMS1117-3.3, U11 AMS1117-5.0, U12 MPU-6050, U2 ACS712xLCTR-30A, U3 ACS712xLCTR-30A, U4 ACS712xLCTR-30A, U5 ACS712xLCTR-30A, U6 ACS712xLCTR-30A, U7 ACS712xLCTR-30A, U8 LM75B

Commit message: Update to v1
Parts:
- added C20: 100nF, Capacitor_SMD:C_0603_1608Metric, F.Cu at (145.9, 56.0)
- added C21: 100nF, Capacitor_SMD:C_0603_1608Metric, F.Cu at (149.8, 60.5)
- added C22: 100nF, Capacitor_SMD:C_0603_1608Metric, F.Cu at (140.7, 58.7)
- added C23: 100nF, Capacitor_SMD:C_0603_1608Metric, F.Cu at (127.8, 58.0)
- added C24: 100nF, Capacitor_SMD:C_0603_1608Metric, F.Cu at (162.6, 46.4)
- added C25: 100nF, Capacitor_SMD:C_0603_1608Metric, F.Cu at (131.4, 46.7)
- added C26: 100nF, Capacitor_SMD:C_0603_1608Metric, F.Cu at (119.0, 48.1)
- added C27: 1uF, Capacitor_SMD:C_0603_1608Metric, F.Cu at (153.0, 96.0)
- added U13: LM75B, Package_SO:SOIC-8_3.9x4.9mm_P1.27mm, F.Cu at (146.1, 107.8)
- added U9: AS5047D, Package_SO:TSSOP-14_4.4x5mm_P0.65mm, F.Cu at (146.6, 100.9)
- C18: value 2.2nF -> 100nF
- U12: value MPU-6050 -> MCP3008; footprint Sensor_Motion:InvenSense_QFN-24_4x4mm_P0.5mm -> Package_SO:SOIC-16_3.9x9.9mm_P1.27mm
- moved C17 27.3 mm to (165.2, 120.0), turned to -90 degrees
- moved U12 22.6 mm to (160.6, 122.4), turned to 0 degrees
- moved C19 4.21 mm to (147.8, 97.3)
- moved C18 3.51 mm to (149.7, 105.8), turned to -90 degrees
Connections:
- C17 pad 1: Net-(U12-REGOUT) -> +5V
- C18 pad 1: Net-(U12-CPOUT) -> +5V
- C19 pad 1: +3.3V -> +5V
- J10 pad 3: ADC6 -> /Logica/ADC1
- J10 pad 4: ADC5 -> /Logica/ADC2
- J10 pad 5: ADC4 -> /Logica/ADC3
- J10 pad 6: ADC3 -> /Logica/ADC4
- J10 pad 7: ADC2 -> /Logica/ADC5
- J10 pad 8: ADC1 -> /Logica/ADC6
- U1 pad 12: ADC2 -> /Logica/CS_ADC
- U1 pad 17: ADC3 -> unconnected-(U1-IO9-Pad17)
- U1 pad 18: ADC4 -> unconnected-(U1-IO10-Pad18)
- U1 pad 19: ADC5 -> unconnected-(U1-IO11-Pad19)
- U1 pad 20: ADC6 -> unconnected-(U1-IO12-Pad20)
- U1 pad 28: unconnected-(U1-IO35-Pad28) -> /Logica/MOSI
- U1 pad 29: unconnected-(U1-IO36-Pad29) -> /Logica/SCK
- U1 pad 30: unconnected-(U1-IO37-Pad30) -> /Logica/MISO
- U1 pad 7: ADC1 -> /Logica/CS_INCL
- U12 pad 1: GND -> /Logica/ADC1
- U12 pad 10: Net-(U12-REGOUT) -> /Logica/CS_ADC
- U12 pad 11: GND -> /Logica/MOSI
- U12 pad 12: unconnected-(U12-INT-Pad12) -> /Logica/MISO
- U12 pad 13: +3.3V -> /Logica/SCK
- U12 pad 14: unconnected-(U12-NC-Pad14) -> GND
- U12 pad 15: unconnected-(U12-NC-Pad15) -> +5V
- U12 pad 16: unconnected-(U12-NC-Pad16) -> +5V
- U12 pad 2: unconnected-(U12-NC-Pad2) -> /Logica/ADC2
- U12 pad 3: unconnected-(U12-NC-Pad3) -> /Logica/ADC3
- U12 pad 4: unconnected-(U12-NC-Pad4) -> /Logica/ADC4
- U12 pad 5: unconnected-(U12-NC-Pad5) -> /Logica/ADC5
- U12 pad 6: unconnected-(U12-AUX_DA-Pad6) -> /Logica/ADC6
- U12 pad 8: +3.3V -> unconnected-(U12-CH7-Pad8)
Routing:
- net /Logica/MISO: track 0.00 -> 67.5 mm, vias 0 -> 4
- net /Logica/MOSI: track 0.00 -> 66.7 mm, vias 0 -> 4
- net /Logica/SCK: track 0.00 -> 64.6 mm, vias 0 -> 4
- net ADC1: track 63.2 -> 0.00 mm, vias 1 -> 0
- net GND: track 276.6 -> 336.0 mm, vias 12 -> 14
- net ADC2: track 54.7 -> 0.00 mm, vias 1 -> 0
- net /Logica/CS_ADC: track 0.00 -> 49.5 mm, vias 0 -> 2
- net ADC6: track 49.1 -> 0.00 mm, vias 1 -> 0
- net ADC3: track 48.9 -> 0.00 mm, vias 2 -> 0
- net ADC4: track 48.7 -> 0.00 mm, vias 2 -> 0
- net ADC5: track 48.4 -> 0.00 mm, vias 1 -> 0
- net /Logica/CS_INCL: track 0.00 -> 41.8 mm, vias 0 -> 2
- net +5V: track 31.9 -> 71.9 mm, vias 1 -> 2
- net GND1: track 245.0 -> 279.7 mm, vias 10 -> 12
- net +5VA: track 97.1 -> 123.8 mm
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Other:
- board text added: "+"
- board text added: "-"
- board text added: "EJE1"
- board text added: "EJE2"
- board text added: "EJE3"

Commit message: Update v1
Changed lines of the file:
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@@
 		)
 		(property "Value" "100nF"
-			(at 0 1.43 90)
+			(at 1.85 -0.09 180)
 			(layer "F.SilkS")
 			(effects
