File: Hardware/PCB/IMPASS/Logica.kicad_sch (KiCad schematic)
At the start: 69 parts, among them J1 PUENTE H, J10 SENSORES, J12 POWER, J7 PUENTE H, J8 SOLENOIDES, J9 PROG, Q25 2N7002, Q26 2N7002, Q27 2N7002, Q28 2N7002, Q29 2N7002, Q30 2N7002, Q31 2N7002, Q32 2N7002, Q33 2N7002, Q34 2N7002, Q35 2N7002, Q36 2N7002, Q37 2N7002, Q38 2N7002, Q39 2N7002, Q40 2N7002, Q41 2N7002, Q42 2N7002, Q46 2N7002, Q47 2N7002, Q48 2N7002, SW1 RESET, SW2 BOOT, U1 ESP32-S3-WROOM-1, U10 AMS1117-3.3, U11 AMS1117-5.0

Commit message: Update to v1
Connections:
- net ADC1: now also J10.3 (Pin_3); no longer J10.8 (Pin_8), U1.7 (IO7)
- net ADC2: now also J10.4 (Pin_4); no longer J10.7 (Pin_7), U1.12 (IO8)
- net ADC3: now also J10.5 (Pin_5); no longer J10.6 (Pin_6), U1.17 (IO9)
- net ADC4: now also J10.6 (Pin_6); no longer J10.5 (Pin_5), U1.18 (IO10)
- net ADC5: now also J10.7 (Pin_7); no longer J10.4 (Pin_4), U1.19 (IO11)
- net ADC6: now also J10.8 (Pin_8); no longer J10.3 (Pin_3), U1.20 (IO12)
- net MOSI: now reaches U1.28 (IO35)
- net SCK: now reaches U1.29 (IO36)
- net MISO: now reaches U1.30 (IO37)
- new net CS_ADC: U1.12 (IO8)
- new net CS_INCL: U1.7 (IO7)
- no-connect marks 10 -> 11

Commit message: Update v1
Other:
- company: (none) -> Luis Miguel Carmona Cortés
- title: (none) -> IMPASS 
Changed lines of the file:
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@@
 	(generator_version "8.0")
 	(paper "A4")
+	(title_block
+		(title "IMPASS ")
+		(date "2026-01-12")
+		(rev "v1.0")
+		(company "Luis Miguel Carmona Cortés")
+		(comment 1 "Lógica electrónica para poder controlar con 2 pines los puentes H")
+		(comment 2 "Connectores para recibir las señales de los sensores")
+		(comment 3 "Progrmación de la ESP32-S3")
+	)
 	(junction
 		(at 102.87 152.4)
