File: Hardware/PCB/IMPASS/Potencia.kicad_sch (KiCad schematic)
At the start: 8 parts, among them J14 SOLENOIDES, J15 PUENTE H, J16 PUENTE H, J2 POWER, J3 EJE1, J4 EJE2, J5 EJE3, J6 VM

Commit message: IMPASS schematics update
Connections:
- net OUT1_1 renamed out1_5
- net OUT1_2 renamed out2_5
- net OUT1_3 renamed out1_3
- net OUT1_4 renamed out2_2
- net OUT1_5 renamed out1_2
- net OUT1_6 renamed out2_4
- net OUT2_1 renamed out2_6
- net OUT2_2 renamed out1_6
- net OUT2_3 renamed out1_4
- net OUT2_4 renamed out2_1
- net OUT2_5 renamed out1_1
- net OUT2_6 renamed out2_3

Commit message: Update v1
Other:
- company: (none) -> Luis Miguel Carmona Cortés
- title: (none) -> IMPASS 
Changed lines of the file:
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@@
 	(generator_version "8.0")
 	(paper "A4")
+	(title_block
+		(title "IMPASS ")
+		(date "2026-01-12")
+		(rev "v1.0")
+		(company "Luis Miguel Carmona Cortés")
+		(comment 1 "Circuitos de potencia")
+	)
 	(junction
 		(at 57.15 76.2)
