File: Hardware/PCB/IMPASS/eje2.kicad_sch (KiCad schematic)
At the start: 8 parts, among them Q10 DMN3008SFG, Q11 DMN3008SFG, Q12 DMN3008SFG, Q13 DMN3008SFG, Q14 DMN3008SFG, Q15 DMN3008SFG, Q16 DMN3008SFG, Q9 DMN3008SFG

Commit message: IMPASS schematics update
Connections:
- net OUT1_4: now also Q10.1 (S), Q10.2 (S), Q10.3 (S), Q12.5 (D); no longer Q13.1 (S), Q13.2 (S), Q13.3 (S), Q15.5 (D)
- net OUT2_3: now also Q13.1 (S), Q13.2 (S), Q13.3 (S), Q15.5 (D); no longer Q10.1 (S), Q10.2 (S), Q10.3 (S), Q12.5 (D)

Commit message: Update v1
Other:
- company: (none) -> Luis Miguel Carmona Cortés
- title: (none) -> IMPASS 
Changed lines of the file:
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@@
 	(generator_version "8.0")
 	(paper "A4")
+	(title_block
+		(title "IMPASS ")
+		(date "2026-01-12")
+		(rev "v1.0")
+		(company "Luis Miguel Carmona Cortés")
+		(comment 1 "Puentes H del eje2")
+	)
 	(junction
 		(at 128.27 39.37)
