File: Hardware/PCB/IMPASS/eje2.kicad_sch (KiCad schematic)
At the start: 8 parts, among them Q10 DMN3008SFG, Q11 DMN3008SFG, Q12 DMN3008SFG, Q13 DMN3008SFG, Q14 DMN3008SFG, Q15 DMN3008SFG, Q16 DMN3008SFG, Q9 DMN3008SFG

Commit message: Hardware: update schematic and PCB layout
Parts:
- removed Q10, Q13, Q14, Q9: DMN3008SFG, Package_SON:Diodes_PowerDI3333-8, symbol Transistor_FET:DMN3008SFG
- added Q10, Q7: BC847BDW1, Package_TO_SOT_SMD:SOT-363_SC-70-6, symbol Transistor_BJT:BC847BDW1
- added Q13, Q14, Q8, Q9: DMP3013SFV, Package_SON:Diodes_PowerDI3333-8, symbol Transistor_FET:DMP3013SFV
- added R67, R68, R69, R70, R71, R72, R73, R74: 10k, Resistor_SMD:R_0603_1608Metric, symbol Device:R
Connections:
- net GND: now also Q10.1 (E1), Q10.4 (E2), Q7.1 (E1), Q7.4 (E2)
- net OUT3_1: now also Q8.5 (D)
- net OUT3_2: now also Q9.5 (D)
- net OUT4_1: now also Q13.5 (D)
- net OUT4_2: now also Q14.5 (D)
- net PWM3: now also R67.1
- net PWM4: now also R71.1
- net Vm: now also Q13.1 (S), Q13.2 (S), Q13.3 (S), Q14.1 (S), Q14.2 (S), Q14.3 (S), Q8.1 (S), Q8.2 (S), Q8.3 (S), Q9.1 (S), Q9.2 (S), Q9.3 (S), R68.1, R69.1, R72.1, R73.1
- net ~PWM3: now also R70.2
- net ~PWM4: now also R74.2
- new net: Q7.6 (C1), Q8.4 (G), R68.2
- new net: Q7.3 (C2), Q9.4 (G), R69.2
- new net: Q10.2 (B1), R71.2
- new net: Q10.3 (C2), Q14.4 (G), R73.2
- new net: Q10.6 (C1), Q13.4 (G), R72.2
- new net: Q7.5 (B2), R70.1
- new net: Q7.2 (B1), R67.2
- new net: Q10.5 (B2), R74.1
