File: Hardware/PCB/IMPASS/eje3.kicad_sch (KiCad schematic)
At the start: 8 parts, among them Q17 DMN3008SFG, Q18 DMN3008SFG, Q19 DMN3008SFG, Q20 DMN3008SFG, Q21 DMN3008SFG, Q22 DMN3008SFG, Q23 DMN3008SFG, Q24 DMN3008SFG

Commit message: Update v1
Other:
- company: (none) -> Luis Miguel Carmona Cortés
- title: (none) -> IMPASS 
Changed lines of the file:
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@@
 	(generator_version "8.0")
 	(paper "A4")
+	(title_block
+		(title "IMPASS ")
+		(date "2026-01-12")
+		(rev "v1.0")
+		(company "Luis Miguel Carmona Cortés")
+		(comment 1 "Puentes H del eje3")
+	)
 	(junction
 		(at 106.68 111.76)
