File: Hardware/PCB/IMPASS/solenoides.kicad_sch (KiCad schematic)
At the start: 7 parts, among them J11 SOLENOIDES, Q43 DMN3008SFG, Q44 DMN3008SFG, Q45 DMN3008SFG

Commit message: IMPASS schematics update
Connections:
- net at J11.1 (Pin_1): now also Q45.4 (G); no longer Q44.4 (G)
- net at J11.3 (Pin_3): now also Q44.4 (G); no longer Q45.4 (G)
Changed lines of the file:
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@@
-	(wire
-		(pts
-			(xy 100.33 59.69) (xy 88.9 59.69)
-		)
-		(stroke
-			(width 0)
-			(type default)
-		)
-	)
-	(wire
-		(pts
-			(xy 88.9 54.61) (xy 109.22 54.61)
-		)
-		(stroke
-			(width 0)
-			(type default)
-		)
-	)
 	(wire
 		(pts
@@
 		(pts
 			(xy 116.84 93.98) (xy 116.84 59.69)
-		)
-		(stroke
-			(width 0)
-			(type default)
-		)
-	)
-	(wire
-		(pts
-			(xy 100.33 87.63) (xy 100.33 59.69)
 		)
 		(stroke
@@
 		(pts
 			(xy 143.51 55.88) (xy 128.27 55.88)
+		)
+		(stroke
+			(width 0)
+			(type default)
+		)
+	)
+	(wire
+		(pts
+			(xy 88.9 57.15) (xy 106.68 57.15)
+		)
+		(stroke
+			(width 0)
+			(type default)
+		)
+	)
+	(wire
+		(pts
+			(xy 88.9 59.69) (xy 109.22 59.69)
 		)
 		(stroke
@@
 	(wire
 		(pts
-			(xy 106.68 57.15) (xy 88.9 57.15)
+			(xy 128.27 55.88) (xy 128.27 41.91)
 		)
 		(stroke
@@
 	(wire
 		(pts
-			(xy 128.27 55.88) (xy 128.27 41.91)
+			(xy 109.22 54.61) (xy 109.22 59.69)
 		)
 		(stroke
+			(width 0)
+			(type default)
+		)
+	)
+	(wire
+		(pts
+			(xy 88.9 54.61) (xy 100.33 54.61)
+		)
+		(stroke
+			(width 0)
+			(type default)
+		)
+	)
+	(wire
+		(pts
+			(xy 100.33 54.61) (xy 100.33 87.63)
+		)
+		(stroke

Commit message: Update v1
Other:
- company: (none) -> Luis Miguel Carmona Cortés
- title: (none) -> IMPASS 
Changed lines of the file:
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@@
 	(generator_version "8.0")
 	(paper "A4")
+	(title_block
+		(title "IMPASS ")
+		(date "2026-01-12")
+		(rev "v1.0")
+		(company "Luis Miguel Carmona Cortés")
+		(comment 1 "Mosfet H de los solenoides")
+	)
 	(junction
 		(at 116.84 49.53)
