File: Hardware/PCB/IMPASS/sensores_potencia.kicad_sch (KiCad schematic)
At the start: 32 parts, among them U2 LM75B, U3 ACS712xLCTR-30A, U4 ACS712xLCTR-30A, U5 ACS712xLCTR-30A, U6 ACS712xLCTR-30A, U7 ACS712xLCTR-30A, U8 ACS712xLCTR-30A

Commit message: Hardware: update schematic and PCB layout
Connections:
- net OUT1_1 renamed IN1_1
- net OUT2_1 renamed IN2_1
- net OUT3_1 renamed IN3_1
- net OUT4_1 renamed IN4_1
- net OUT5_1 renamed IN5_1
- net OUT6_1 renamed IN6_1
