File: Hardware/PCB/IMPASS/sensores_potencia.kicad_sch (KiCad schematic)
At the start: 32 parts, among them U2 LM75B, U3 ACS712xLCTR-30A, U4 ACS712xLCTR-30A, U5 ACS712xLCTR-30A, U6 ACS712xLCTR-30A, U7 ACS712xLCTR-30A, U8 ACS712xLCTR-30A

Commit message: Hardware: Update all the logic pcb 	- added ads1015 	- added the logic foe P-MOSFET 	- added I2C connector
Parts:
- removed D1, D2, D3, D4, D5, D6: 1N4448, Diode_THT:D_DO-35_SOD27_P2.54mm_Vertical_AnodeUp, symbol Diode:1N4448
- removed R21, R22, R23, R24, R25, R26: 2k, Resistor_SMD:R_0603_1608Metric, symbol Device:R
Connections:
- net I_1: now also U3.7 (VIOUT)
- net I_2: now also U4.7 (VIOUT)
- net I_3: now also U5.7 (VIOUT)
- net I_4: now also U6.7 (VIOUT)
- net I_5: now also U7.7 (VIOUT)
- net I_6: now also U8.7 (VIOUT)
