File: Hardware/PCB/IMPASS/IMPASS.kicad_sch (KiCad schematic)
At the start: 15 parts, among them J1 POWER, U1 TPS62162DSG, U15 TPS62163DSG

Commit message: Hardware: Update all the logic pcb 	- added ads1015 	- added the logic foe P-MOSFET 	- added I2C connector
Parts:
- removed D8, D9: LED, LED_SMD:LED_0603_1608Metric, symbol Device:LED
- removed R34, R85: 100, Resistor_SMD:R_0603_1608Metric, symbol Device:R
Connections:
- net 12v renamed +12V
