File: Hardware/PCB/IMPASS/placa_potencia.kicad_sch (KiCad schematic)
At the start: 15 parts, among them J11 SOLENOIDES, J2 POWER, J22 VM, J23 EJE1, J24 EJE2, J25 EJE3, J26 SOLENOIDES, J27 PUENTE H, J28 PUENTE H, J29 SENSORES

Commit message: Hardware: Update all the logic pcb 	- added ads1015 	- added the logic foe P-MOSFET 	- added I2C connector
Parts:
- removed D7: SS14, Diode_SMD:D_SMA, symbol Diode:SS14
Changed lines of the file:
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@@
 		(comment 2 "Esta es la placa de potencia")
 	)
-	(junction
-		(at 45.72 20.32)
-		(diameter 0)
-		(color 0 0 0 0)
-	)
-	(junction
-		(at 45.72 17.78)
-		(diameter 0)
-		(color 0 0 0 0)
-	)
 	(wire
 		(pts
@@
 	(wire
 		(pts
-			(xy 50.8 15.24) (xy 46.99 15.24)
-		)
-		(stroke
-			(width 0)
-			(type default)
-		)
-	)
-	(wire
-		(pts
 			(xy 148.59 29.21) (xy 152.4 29.21)
 		)
@@
 	(wire
 		(pts
-			(xy 48.26 20.32) (xy 45.72 20.32)
-		)
-		(stroke
-			(width 0)
-			(type default)
-		)
-	)
-	(wire
-		(pts
 			(xy 152.4 68.58) (xy 153.67 68.58)
 		)
@@
 	(wire
 		(pts
-			(xy 46.99 17.78) (xy 45.72 17.78)
-		)
-		(stroke
-			(width 0)
-			(type default)
-		)
-	)
-	(wire
-		(pts
 			(xy 67.31 91.44) (xy 71.12 91.44)
 		)
@@
 	(wire
 		(pts
-			(xy 48.26 22.86) (xy 48.26 20.32)
-		)
-		(stroke
-			(width 0)
-			(type default)
-		)
-	)
-	(wire
-		(pts
 			(xy 151.13 81.28) (xy 151.13 104.14)
 		)
@@
 	(wire
 		(pts
-			(xy 46.99 15.24) (xy 46.99 17.78)
-		)
-		(stroke
-			(width 0)
-			(type default)
-		)
-	)
-	(wire
-		(pts
 			(xy 97.79 92.71) (xy 102.87 92.71)
 		)
@@
 	(wire
 		(pts
-			(xy 50.8 22.86) (xy 48.26 22.86)
-		)
-		(stroke
-			(width 0)
-			(type default)
-		)
-	)
-	(wire
-		(pts
 			(xy 69.85 93.98) (xy 67.31 93.98)
 		)
@@
 					(unit 1)
 				)
-			)
-		)
-	)
-	(symbol
-		(lib_id "Diode:SS14")
-		(at 50.8 19.05 270)
-		(unit 1)
-		(body_style 1)
-		(exclude_from_sim no)
-		(in_bom yes)
-		(on_board yes)
-		(in_pos_files yes)
-		(dnp no)
-		(fields_autoplaced yes)
-		(property "Reference" "D7"
-			(at 53.34 17.4624 90)
-			(show_name no)
-			(do_not_autoplace no)
-			(effects
-				(font
-					(size 1.27 1.27)
-				)
-				(justify left)
-			)
-		)
-		(property "Value" "SS14"
-			(at 53.34 20.0024 90)
-			(show_name no)
-			(do_not_autoplace no)
-			(effects
-				(font
-					(size 1.27 1.27)
-				)
-				(justify left)
-			)
-		)
-		(property "Footprint" "Diode_SMD:D_SMA"
-			(at 46.355 19.05 0)
-			(hide yes)
-			(show_name no)
-			(do_not_autoplace no)
-			(effects
-				(font
-					(size 1.27 1.27)
-				)
-			)
-		)
-		(property "Datasheet" "https://www.vishay.com/docs/88746/ss12.pdf"
-			(at 50.8 19.05 0)
-			(hide yes)
-			(show_name no)
-			(do_not_autoplace no)
-			(effects
-				(font
-					(size 1.27 1.27)
-				)
-			)
-		)
-		(property "Description" "40V 1A Schottky Diode, SMA"
-			(at 50.8 19.05 0)
-			(hide yes)
-			(show_name no)
-			(do_not_autoplace no)
-			(effects
-				(font
-					(size 1.27 1.27)
-				)
-			)
-		)
-		(pin "2"
-		)
-		(pin "1"
-		)
-		(instances
-			(project "IMPASS"
-				(path "/731b3037-3e9a-4423-b2c0-b5bf223d88c2/acd98061-6367-4cb8-aa42-1ec0ef88ad06"
-					(reference "D7")
-					(unit 1)
-				)

Commit message: Hardware: Update all the power pcb 	- added thr MOSFETs         - added the current sensors         - added the lm75 sensor
Connections:
- net Eje3/OUT5_2: now also J25.1 (Pin_1); no longer J25.3 (Pin_3)
- net Eje3/OUT6_2: now also J25.3 (Pin_3); no longer J25.1 (Pin_1)
- net Sensores_potencia/OUT5_2: now also J25.2 (Pin_2); no longer J25.4 (Pin_4)
- net Sensores_potencia/OUT6_2: now also J25.4 (Pin_4); no longer J25.2 (Pin_2)
